File: motor_controller/hardware/motor_controller.kicad_pcb (KiCad board)
At the start: 2 copper layers, 251.5 x 106.7 mm, 57 parts, among them J1 STM32F4_Discovery_Header, J10 Conn_01x02_Male, J11 Conn_01x02_Male, J12 Conn_01x03_Male, J13 Conn_01x06_Male, J14 Conn_01x02_Male, J15 Conn_01x02_Male, J16 pololu-D24V10F5, J17 Conn_01x02_Male, J2 Conn_01x02_Male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

Commit message: Fix fan mounting hole positions
Parts:
- moved MH10 2.54 mm to (223.4, 142.2)
- moved MH7 2.54 mm to (151.9, 70.7)
- moved MH8 2.54 mm to (151.9, 142.2)
- moved MH9 2.54 mm to (223.4, 70.7)
Changed lines of the file:
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@@
     (mod_text_size 1 1)
     (mod_text_width 0.15)
-    (pad_size 1.524 1.524)
-    (pad_drill 0.762)
+    (pad_size 3.2 3.2)
+    (pad_drill 3.2)
     (pad_to_mask_clearance 0.2)
     (aux_axis_origin 0 0)
@@
   )
   (module MountingHole:MountingHole_3.2mm_M3_DIN965 (layer F.Cu)
-    (at 149.35 70.74)
+    (at 151.89 70.74)
     (descr "Mounting Hole 3.2mm, no annular, M3, DIN965")
     (tags "mounting hole 3.2mm no annular m3 din965")
@@
   )
   (module MountingHole:MountingHole_3.2mm_M3_DIN965 (layer F.Cu)
-    (at 149.35 142.24)
+    (at 151.89 142.24)
     (descr "Mounting Hole 3.2mm, no annular, M3, DIN965")
     (tags "mounting hole 3.2mm no annular m3 din965")
@@
     (fp_circle (center 0 0) (end 2.8 0) (layer Cmts.User) (width 0.15))
     (fp_circle (center 0 0) (end 3.05 0) (layer F.CrtYd) (width 0.05))
-    (pad 1 np_thru_hole circle (at 0 0) (size 3.2 3.2) (drill 3.2) (layers *.Cu *.Mask))
+    (pad "" np_thru_hole circle (at 0 0) (size 3.2 3.2) (drill 3.2) (layers *.Cu *.Mask)
+      (clearance 1.27))
   )
   (module MountingHole:MountingHole_3.2mm_M3_DIN965 (layer F.Cu)
-    (at 220.85 70.74)
+    (at 223.39 70.74)
     (descr "Mounting Hole 3.2mm, no annular, M3, DIN965")
     (tags "mounting hole 3.2mm no annular m3 din965")
@@
   )
   (module MountingHole:MountingHole_3.2mm_M3_DIN965 (layer F.Cu)
-    (at 220.85 142.24)
+    (at 223.39 142.24)
     (descr "Mounting Hole 3.2mm, no annular, M3, DIN965")
     (tags "mounting hole 3.2mm no annular m3 din965")
@@
       (pts
         (xy 268.732 50.8) (xy 130.81 50.8) (xy 130.81 76.2) (xy 251.46 76.2) (xy 251.46 135.89)
-        (xy 154.305 135.89) (xy 154.305 162.56) (xy 269.24 162.56) (xy 269.24 50.8)
+        (xy 155.575 135.89) (xy 155.575 162.56) (xy 269.24 162.56) (xy 269.24 50.8)
       )
     )
@@
       (pts
         (xy 12.7 50.8) (xy 129.54 50.8) (xy 129.54 77.47) (xy 250.19 77.47) (xy 250.19 134.62)
-        (xy 153.035 134.62) (xy 153.035 162.56) (xy 12.7 162.56)
+        (xy 154.305 134.62) (xy 154.305 162.56) (xy 12.7 162.56)
       )
     )

Commit message: Add transient protection for motors
Parts:
- added C12: C, Capacitor_SMD:C_1206_3216Metric_Pad1.42x1.75mm_HandSolder, B.Cu at (235.6, 56.5)
- added C13: C, Capacitor_SMD:C_1206_3216Metric_Pad1.42x1.75mm_HandSolder, B.Cu at (199.4, 56.5)
- added C14: C, Capacitor_SMD:C_1206_3216Metric_Pad1.42x1.75mm_HandSolder, B.Cu at (163.4, 56.5)
- added C15: C, Capacitor_SMD:C_1206_3216Metric_Pad1.42x1.75mm_HandSolder, B.Cu at (169.5, 155.6)
- added C16: C, Capacitor_SMD:C_1206_3216Metric_Pad1.42x1.75mm_HandSolder, B.Cu at (206.2, 155.6)
- added C17: C, Capacitor_SMD:C_1206_3216Metric_Pad1.42x1.75mm_HandSolder, B.Cu at (242.4, 155.6)
- added D1: DIODE, Diode_SMD:D_SMB_Handsoldering, B.Cu at (259.2, 83.8)
- added D10: DIODE, Diode_SMD:D_SMB_Handsoldering, F.Cu at (154.3, 61.0)
- added D11: DIODE, Diode_SMD:D_SMB_Handsoldering, B.Cu at (154.5, 61.0)
- added D12: DIODE, Diode_SMD:D_SMB_Handsoldering, F.Cu at (179.1, 61.0)
- added D13: DIODE, Diode_SMD:D_SMB_Handsoldering, B.Cu at (179.1, 61.0)
- added D14: DIODE, Diode_SMD:D_SMB_Handsoldering, F.Cu at (179.5, 151.1)
- added D15: DIODE, Diode_SMD:D_SMB_Handsoldering, B.Cu at (179.7, 151.1)
- added D16: DIODE, Diode_SMD:D_SMB_Handsoldering, F.Cu at (154.3, 151.1)
- added D17: DIODE, Diode_SMD:D_SMB_Handsoldering, B.Cu at (154.3, 151.1)
- added D18: DIODE, Diode_SMD:D_SMB_Handsoldering, F.Cu at (215.3, 151.1)
- added D19: DIODE, Diode_SMD:D_SMB_Handsoldering, B.Cu at (215.4, 151.1)
- added D2: DIODE, Diode_SMD:D_SMB_Handsoldering, F.Cu at (226.7, 61.0)
- added D20: DIODE, Diode_SMD:D_SMB_Handsoldering, F.Cu at (190.3, 151.1)
- added D21: DIODE, Diode_SMD:D_SMB_Handsoldering, B.Cu at (190.3, 151.1)
- added D22: DIODE, Diode_SMD:D_SMB_Handsoldering, F.Cu at (251.5, 151.1)
- added D23: DIODE, Diode_SMD:D_SMB_Handsoldering, B.Cu at (251.5, 151.1)
- added D24: DIODE, Diode_SMD:D_SMB_Handsoldering, F.Cu at (226.2, 151.1)
- added D25: DIODE, Diode_SMD:D_SMB_Handsoldering, B.Cu at (226.2, 151.1)
- added D3: DIODE, Diode_SMD:D_SMB_Handsoldering, B.Cu at (226.7, 61.0)
- added D4: DIODE, Diode_SMD:D_SMB_Handsoldering, F.Cu at (250.8, 61.0)
- added D5: DIODE, Diode_SMD:D_SMB_Handsoldering, B.Cu at (250.8, 61.0)
- added D6: DIODE, Diode_SMD:D_SMB_Handsoldering, F.Cu at (190.3, 61.0)
- added D7: DIODE, Diode_SMD:D_SMB_Handsoldering, B.Cu at (190.3, 61.0)
- added D8: DIODE, Diode_SMD:D_SMB_Handsoldering, F.Cu at (215.3, 61.0)
- added D9: DIODE, Diode_SMD:D_SMB_Handsoldering, B.Cu at (215.3, 61.0)
- added R10: R, Resistor_SMD:R_1206_3216Metric_Pad1.42x1.75mm_HandSolder, B.Cu at (163.6, 155.6)
- added R11: R, Resistor_SMD:R_1206_3216Metric_Pad1.42x1.75mm_HandSolder, B.Cu at (199.6, 155.6)
- added R12: R, Resistor_SMD:R_1206_3216Metric_Pad1.42x1.75mm_HandSolder, B.Cu at (235.8, 155.6)
- added R7: R, Resistor_SMD:R_1206_3216Metric_Pad1.42x1.75mm_HandSolder, B.Cu at (242.2, 56.5)
- added R8: R, Resistor_SMD:R_1206_3216Metric_Pad1.42x1.75mm_HandSolder, B.Cu at (205.7, 56.5)
- added R9: R, Resistor_SMD:R_1206_3216Metric_Pad1.42x1.75mm_HandSolder, B.Cu at (169.8, 56.5)
- moved C10 1.91 mm to (260.4, 69.2)
- moved C11 0.75 mm to (260.4, 135.4)
Routing:
- net Net-(C15-Pad2): track 10.7 -> 30.3 mm
- net Net-(C13-Pad2): track 10.6 -> 30.0 mm
- net Net-(D12-Pad1): track 10.6 -> 30.0 mm
- net Net-(C17-Pad2): track 10.9 -> 30.3 mm
- net Net-(D24-Pad1): track 10.9 -> 30.1 mm
- net Net-(D8-Pad1): track 10.6 -> 29.6 mm
- net Net-(D16-Pad1): track 10.7 -> 29.7 mm
- net Net-(C12-Pad2): track 10.7 -> 29.6 mm
- net Net-(C14-Pad2): track 10.6 -> 29.2 mm
- net Net-(D4-Pad1): track 10.7 -> 29.2 mm
- net Net-(D20-Pad1): track 10.9 -> 22.9 mm
- net Net-(C16-Pad2): track 10.9 -> 22.7 mm
- net +24V: track 13.3 -> 17.7 mm
- net Net-(C12-Pad1): track 0.00 -> 3.59 mm
- net Net-(C17-Pad1): track 0.00 -> 3.58 mm
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
Commit message: Add protection for motor controller GND
Parts:
- added L3: Ferrite_Bead_Small, Inductor_SMD:L_0805_2012Metric_Pad1.15x1.40mm_HandSolder, F.Cu at (247.0, 104.5)
- added L4: Ferrite_Bead_Small, Inductor_SMD:L_0805_2012Metric_Pad1.15x1.40mm_HandSolder, F.Cu at (217.6, 100.3)
- added L5: Ferrite_Bead_Small, Inductor_SMD:L_0805_2012Metric_Pad1.15x1.40mm_HandSolder, F.Cu at (180.3, 98.8)
- added L6: Ferrite_Bead_Small, Inductor_SMD:L_0805_2012Metric_Pad1.15x1.40mm_HandSolder, F.Cu at (153.7, 113.4)
- added L7: Ferrite_Bead_Small, Inductor_SMD:L_0805_2012Metric_Pad1.15x1.40mm_HandSolder, F.Cu at (185.7, 112.4)
- added L8: Ferrite_Bead_Small, Inductor_SMD:L_0805_2012Metric_Pad1.15x1.40mm_HandSolder, F.Cu at (223.8, 111.8)
- moved R4 1.66 mm to (152.4, 117.5), turned to 180 degrees
Connections:
- U1 pad 8: GND -> Net-(L3-Pad1)
- U2 pad 8: GND -> Net-(L4-Pad1)
- U3 pad 8: GND -> Net-(L5-Pad1)
- U4 pad 8: GND -> Net-(L6-Pad1)
- U5 pad 8: GND -> Net-(L7-Pad1)
- U6 pad 8: GND -> Net-(L8-Pad1)
Routing:
- net Net-(L7-Pad1): track 0.00 -> 7.44 mm
- net Net-(L8-Pad1): track 0.00 -> 5.17 mm
- net Net-(L5-Pad1): track 0.00 -> 5.09 mm
- net Net-(L4-Pad1): track 0.00 -> 4.86 mm
- net motor_sleep_all: track 223.1 -> 227.8 mm
- net Net-(L6-Pad1): track 0.00 -> 4.17 mm
- net Net-(L3-Pad1): track 0.00 -> 3.61 mm
- net motor_pwm_4: track 80.9 -> 83.6 mm
- net Net-(R4-Pad2): track 5.38 -> 7.52 mm
- net motor_fault_2: track 120.4 -> 122.2 mm
- net motor_dir_4: track 73.7 -> 74.9 mm
- net motor_current_5: track 185.3 -> 186.5 mm
- net motor_current_6: track 221.4 -> 222.6 mm
- net motor_pwm_5: track 128.6 -> 129.7 mm
- net motor_dir_5: track 113.2 -> 112.5 mm
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Other:
- net class 3-5VSignal added: clearance 0.2, trace_width 0.5, via_dia 1, via_drill 0.6

Commit message: Add optional protection for analog inputs
Parts:
- added C18: C, Capacitor_SMD:C_0805_2012Metric_Pad1.15x1.40mm_HandSolder, B.Cu at (38.1, 111.3)
- added C19: C, Capacitor_SMD:C_0805_2012Metric_Pad1.15x1.40mm_HandSolder, B.Cu at (38.1, 126.2)
- added C20: C, Capacitor_SMD:C_0805_2012Metric_Pad1.15x1.40mm_HandSolder, B.Cu at (38.1, 141.2)
- added C21: C, Capacitor_SMD:C_0805_2012Metric_Pad1.15x1.40mm_HandSolder, B.Cu at (38.1, 118.9)
- added C22: C, Capacitor_SMD:C_0805_2012Metric_Pad1.15x1.40mm_HandSolder, B.Cu at (38.1, 133.6)
- added C23: C, Capacitor_SMD:C_0805_2012Metric_Pad1.15x1.40mm_HandSolder, B.Cu at (38.1, 148.8)
- added L10: Ferrite, Inductor_SMD:L_0805_2012Metric_Pad1.15x1.40mm_HandSolder, B.Cu at (37.9, 99.1)
- added L11: Ferrite, Inductor_SMD:L_0805_2012Metric_Pad1.15x1.40mm_HandSolder, B.Cu at (38.1, 121.3)
- added L12: Ferrite, Inductor_SMD:L_0805_2012Metric_Pad1.15x1.40mm_HandSolder, B.Cu at (38.1, 113.8)
- added L13: Ferrite, Inductor_SMD:L_0805_2012Metric_Pad1.15x1.40mm_HandSolder, B.Cu at (38.1, 136.1)
- added L14: Ferrite, Inductor_SMD:L_0805_2012Metric_Pad1.15x1.40mm_HandSolder, B.Cu at (38.1, 128.9)
- added L15: Ferrite, Inductor_SMD:L_0805_2012Metric_Pad1.15x1.40mm_HandSolder, B.Cu at (38.1, 151.6)
- added L16: Ferrite, Inductor_SMD:L_0805_2012Metric_Pad1.15x1.40mm_HandSolder, B.Cu at (38.1, 143.9)
- added L9: Ferrite, Inductor_SMD:L_0805_2012Metric_Pad1.15x1.40mm_HandSolder, B.Cu at (37.9, 104.1)
- added TP1: TestPoint, TestPoint:TestPoint_Pad_D1.0mm, F.Cu at (20.3, 104.1)
- added TP2: TestPoint, TestPoint:TestPoint_Pad_D1.0mm, F.Cu at (20.3, 99.1)
- added TP3: TestPoint, TestPoint:TestPoint_Pad_D1.0mm, F.Cu at (20.6, 121.3)
- added TP4: TestPoint, TestPoint:TestPoint_Pad_D1.0mm, F.Cu at (20.6, 116.8)
- added TP5: TestPoint, TestPoint:TestPoint_Pad_D1.0mm, F.Cu at (20.6, 134.0)
- added TP6: TestPoint, TestPoint:TestPoint_Pad_D1.0mm, F.Cu at (20.6, 129.5)
- added TP7: TestPoint, TestPoint:TestPoint_Pad_D1.0mm, F.Cu at (20.6, 146.7)
- added TP8: TestPoint, TestPoint:TestPoint_Pad_D1.0mm, F.Cu at (20.6, 142.2)
Connections:
- J1 pad 11: motor_pot_2 -> motor_pot_1
- J1 pad 13: motor_pot_3 -> motor_pot_4
- J1 pad 15: motor_pot_4 -> motor_pot_3
- J1 pad 19: motor_pot_5 -> motor_pot_6
- J1 pad 21: motor_pot_6 -> motor_pot_5
- J1 pad 7: motor_pot_1 -> motor_pot_2
- J10 pad 1: motor_pot_3 -> Net-(J10-Pad1)
- J10 pad 2: motor_pot_4 -> Net-(J10-Pad2)
- J11 pad 1: motor_pot_5 -> Net-(J11-Pad1)
- J11 pad 2: motor_pot_6 -> Net-(J11-Pad2)
- J15 pad 1: POT+ -> Net-(J15-Pad1)
- J15 pad 2: GND -> Net-(J15-Pad2)
- J9 pad 1: motor_pot_1 -> Net-(J9-Pad1)
- J9 pad 2: motor_pot_2 -> Net-(J9-Pad2)
Routing:
- net uart_rx: track 71.8 -> 92.6 mm
- net Net-(J11-Pad1): track 0.00 -> 19.5 mm
- net Net-(J9-Pad2): track 0.00 -> 17.8 mm
- net Net-(J11-Pad2): track 0.00 -> 17.7 mm
- net Net-(J10-Pad1): track 0.00 -> 17.4 mm
- net Net-(J10-Pad2): track 0.00 -> 16.8 mm
- net Net-(J15-Pad2): track 0.00 -> 16.5 mm
- net Net-(J9-Pad1): track 0.00 -> 16.5 mm
- net Net-(J15-Pad1): track 0.00 -> 15.9 mm
- net uart_tx: track 77.4 -> 90.9 mm
- net motor_pot_1: track 31.0 -> 19.8 mm
- net motor_pot_3: track 36.3 -> 29.6 mm
- net POT+: track 19.1 -> 23.8 mm
- net motor_pot_5: track 41.4 -> 37.5 mm
- net motor_pot_6: track 30.8 -> 32.3 mm
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Other:
- net class Analog: clearance 0.6 -> 0.4; trace_width 1 -> 0.6

Commit message: Add ceramic capacitors into 24V rail
Parts:
- added C24: C, Capacitor_SMD:C_1206_3216Metric_Pad1.42x1.75mm_HandSolder, B.Cu at (227.8, 73.9)
- added C25: C, Capacitor_SMD:C_1206_3216Metric_Pad1.42x1.75mm_HandSolder, B.Cu at (227.8, 67.9)
- added C26: C, Capacitor_SMD:C_1206_3216Metric_Pad1.42x1.75mm_HandSolder, B.Cu at (190.0, 68.6)
- added C27: C, Capacitor_SMD:C_1206_3216Metric_Pad1.42x1.75mm_HandSolder, B.Cu at (190.0, 72.6)
- added C28: C, Capacitor_SMD:C_1206_3216Metric_Pad1.42x1.75mm_HandSolder, B.Cu at (156.0, 73.6)
- added C29: C, Capacitor_SMD:C_1206_3216Metric_Pad1.42x1.75mm_HandSolder, B.Cu at (156.0, 67.9)
- added C30: C, Capacitor_SMD:C_1206_3216Metric_Pad1.42x1.75mm_HandSolder, B.Cu at (179.4, 143.3)
- added C31: C, Capacitor_SMD:C_1206_3216Metric_Pad1.42x1.75mm_HandSolder, B.Cu at (179.4, 139.7)
- added C32: C, Capacitor_SMD:C_1206_3216Metric_Pad1.42x1.75mm_HandSolder, B.Cu at (215.2, 143.3)
- added C33: C, Capacitor_SMD:C_1206_3216Metric_Pad1.42x1.75mm_HandSolder, B.Cu at (215.2, 139.7)
- added C34: C, Capacitor_SMD:C_1206_3216Metric_Pad1.42x1.75mm_HandSolder, B.Cu at (251.7, 143.3)
- added C35: C, Capacitor_SMD:C_1206_3216Metric_Pad1.42x1.75mm_HandSolder, B.Cu at (251.7, 139.7)
- C10, C11: footprint Capacitor_THT:CP_Radial_D18.0mm_P7.50mm -> Capacitor_THT:CP_Radial_D16.0mm_P7.50mm
- moved C10 1.42 mm to (259.1, 69.8)
- moved C11 1.30 mm to (259.1, 135.6)
- moved D1 0.38 mm to (259.1, 84.2)
Routing:
- net +24V: track 17.7 -> 60.0 mm
- net Net-(D20-Pad1): track 22.9 -> 30.2 mm
- net Net-(C16-Pad2): track 22.7 -> 29.8 mm
- net +5V: track 177.7 -> 182.4 mm
